Commit message: 3 robots side by side, only one ball

File: urdf/seveneffort2_across.urdf (robot description, URDF)
Before this commit: robot sevenbot4, 30 links, 29 joints
Joints:
- joint theta1: origin xyz=2 0 0.6 rpy=0 0 0 -> xyz=1 3.5 0.6 rpy=0 0 3.14

File: urdf/seveneffort2_r2.urdf (robot description, URDF)
Before this commit: robot sevenbot2, 30 links, 29 joints
Joints:
- joint theta1: origin xyz=2 0 0.6 rpy=0 0 0 -> xyz=1.5 0 0.6 rpy=0 0 0

File: urdf/seveneffort2_r3.urdf (robot description, URDF)
Before this commit: robot sevenbot3, 30 links, 29 joints
Joints:
- joint theta1: origin xyz=1 3.5 0.6 rpy=0 0 3.14 -> xyz=3 0 0.6 rpy=0 0 0
