Commit message: Set up 3-paddle, 2-ball demo is working with multi-threaded approach, but execution doesnt work well with incorrect hitting velocities

File: urdf/seveneffort2_r2.urdf (robot description, URDF)
Before this commit: robot sevenbot2, 30 links, 29 joints
Joints:
- joint theta1: origin xyz=1.5 0 0.6 rpy=0 0 0 -> xyz=2 0 0.6 rpy=0 0 0
